Commit message: Mod urdf

File: Solver/solver_description/urdf/solver.xacro (robot description, xacro)
@@ -28,13 +28,15 @@
       </visual>
     </link>
-    <link name="imu">
-      <visual>
-        <origin xyz="0 0 0.0" rpy="0 0 0"/>
-          <material name="black"/>
-          <geometry>
-            <box size="0.01 0.01 0.01"/>
-          </geometry>
-      </visual>
-    </link>
+ <link name="imu_link">
+    <visual>
+      <origin rpy="0 0 0" xyz="0 0 0"/>
+      <geometry>
+        <box size="0.033 0.044 0.013"/>
+      </geometry>
+      <material name="xsens_orange">
+        <color rgba="0.92 0.45 0.02 1.0"/>
+      </material>
+    </visual>
+  </link>
     <link name="head_camera">
       <visual>
@@ -48,5 +50,5 @@
     <link name="front/odom">
         <visual>
-            <origin xyz="0 0 0.0" rpy="0 0 0"/>
+            <origin xyz="0 0 0.0" rpy="0 0 0.17"/>
             <material name="black">
             </material>
@@ -76,7 +78,7 @@
     <!-- join between chassi and imu links-->
     <joint name="base_link__imu_link" type="fixed">
-      <origin rpy="0 0 3.14" xyz="-0.094 -0.049 0.1375"/>
+      <origin rpy="0 0 0" xyz="0.20 0 0.29"/>
       <parent link="base_link"/>
-      <child link="imu"/>
+      <child link="imu_link"/>
     </joint>
     <!-- join between chassi and imu links-->

Commit message: MOD urdf

File: Solver/solver_description/urdf/solver.xacro (robot description, xacro)
@@ -32,5 +32,5 @@
       <origin rpy="0 0 0" xyz="0 0 0"/>
       <geometry>
-        <box size="0.033 0.044 0.013"/>
+        <box size="0.044 0.033 0.013"/>
       </geometry>
       <material name="xsens_orange">
